Commit message: feat: update URDF config - 29-DOF G1 robot description with revised inertials and collision geometry

File: src/g1_perception/config/g1_29dof.urdf (robot description, URDF)
Before this commit: robot g1_29dof_rev_1_0, 57 links, 56 joints
Links:
- added link chest_d435_link
Joints:
- added joint chest_d435_joint: type fixed, parent torso_link, child chest_d435_link, origin xyz=0.12875 0.0175 0.165 rpy=0 0 0
